File: ledcube_stick.sch (KiCad schematic (older format))
At the start: 11 parts, among them P1 CONN_02X02, P2 CONN_02X02

Commit message: Detail fix
Other:
- note added: "VDD DRET\nGND DIN"
Changed lines of the file:
@@
 	1250 2650 1250 2875
 Text Notes 8050 2675 0    60   ~ 0
-VDD DRET\nGND DOUT
+VDD DRET\nGND DIN
 $Comp
 L CONN_02X02 P2
